File: H_bridge.kicad_sch (KiCad schematic)
At the start: 11 parts, among them CN1 B6B-PH-K-S(LF)(SN), U13 DRV8870DDA

Commit message: added more symbols
Connections:
- net GND: no longer CN1.2
- net +3.3V renamed ENC_PWR_1
- new net ENC_PWR_2: CN1.2
Changed lines of the file:
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@@
-    (stroke (width 0) (type default))
-  )
-  (wire (pts (xy 138.43 74.93) (xy 152.4 74.93))
-    (stroke (width 0) (type default))
-  )
-  (wire (pts (xy 138.43 90.17) (xy 152.4 90.17))
     (stroke (width 0) (type default))
   )
@@
     (stroke (width 0) (type default))
   )
+  (wire (pts (xy 148.59 90.17) (xy 152.4 90.17))
+    (stroke (width 0) (type default))
+  )
   (wire (pts (xy 100.33 71.12) (xy 100.33 88.9))
     (stroke (width 0) (type default))
@@
     (stroke (width 0) (type default))
   )
+  (wire (pts (xy 148.59 74.93) (xy 152.4 74.93))
+    (stroke (width 0) (type default))
+  )
   (wire (pts (xy 67.31 101.6) (xy 67.31 102.87))
     (stroke (width 0) (type default))
@@
   )
   (wire (pts (xy 113.03 93.98) (xy 113.03 100.33))
-    (stroke (width 0) (type default))
-  )
-  (wire (pts (xy 138.43 63.5) (xy 138.43 74.93))
     (stroke (width 0) (type default))
   )
@@
     (effects (font (size 1.27 1.27)) (justify left bottom))
   )
+  (global_label "ENC_PWR_2" (shape input) (at 148.59 90.17 180) (fields_autoplaced)
+    (effects (font (size 1.27 1.27)) (justify right))
+    (property "Intersheetrefs" "${INTERSHEET_REFS}" (at 134.7986 90.17 0)
+      (effects (font (size 1.27 1.27)) (justify right) hide)
+    )
+  )
+  (global_label "ENC_PWR_1" (shape input) (at 148.59 74.93 180) (fields_autoplaced)
+    (effects (font (size 1.27 1.27)) (justify right))
+    (property "Intersheetrefs" "${INTERSHEET_REFS}" (at 134.7986 74.93 0)
+      (effects (font (size 1.27 1.27)) (justify right) hide)
+    )
+  )
   (hierarchical_label "ENCODER2" (shape output) (at 148.59 80.01 180) (fields_autoplaced)
     (effects (font (size 1.27 1.27)) (justify right))
@@
         (path "/23ba0750-4a55-4d50-828b-749cc0fbb8c8/0734ecc9-bf55-4847-b598-21bbdec71699"
           (reference "#PWR05") (unit 1)
-        )
-      )
-    )
-  )
-  (symbol (lib_id "power:+3.3V") (at 138.43 63.5 0) (unit 1)
-    (in_bom yes) (on_board yes) (dnp no) (fields_autoplaced)
-    (property "Reference" "#PWR0204" (at 138.43 67.31 0)
-      (effects (font (size 1.27 1.27)) hide)
-    )
-    (property "Value" "+3.3V" (at 138.43 59.69 0)
-      (effects (font (size 1.27 1.27)))
-    )
-    (property "Footprint" "" (at 138.43 63.5 0)
-      (effects (font (size 1.27 1.27)) hide)
-    )
-    (property "Datasheet" "" (at 138.43 63.5 0)
-      (effects (font (size 1.27 1.27)) hide)
-    )
-    (pin "1")
-    (instances
-      (project "version_1"
-        (path "/23ba0750-4a55-4d50-828b-749cc0fbb8c8/79f7122c-c2a5-4829-b847-ff54a5199600"
-          (reference "#PWR0204") (unit 1)
-        )
-        (path "/23ba0750-4a55-4d50-828b-749cc0fbb8c8/d2110296-333c-46f5-b5da-c8cbeafe02ed"
-          (reference "#PWR0205") (unit 1)
-        )
-        (path "/23ba0750-4a55-4d50-828b-749cc0fbb8c8/1b8f704b-b129-4c22-a423-d346d579d0e5"
-          (reference "#PWR0206") (unit 1)
-        )
-        (path "/23ba0750-4a55-4d50-828b-749cc0fbb8c8/0734ecc9-bf55-4847-b598-21bbdec71699"
-          (reference "#PWR0207") (unit 1)
         )
       )
@@
         )
       )
-    )
-  )
-  (symbol (lib_id "power:GND") (at 138.43 90.17 0) (mirror y) (unit 1)
-    (in_bom yes) (on_board yes) (dnp no) (fields_autoplaced)
-    (property "Reference" "#PWR010" (at 138.43 96.52 0)
-      (effects (font (size 1.27 1.27)) hide)
-    )
-    (property "Value" "GND" (at 138.43 94.615 0)
-      (effects (font (size 1.27 1.27)))
-    )
-    (property "Footprint" "" (at 138.43 90.17 0)
-      (effects (font (size 1.27 1.27)) hide)
-    )
-    (property "Datasheet" "" (at 138.43 90.17 0)
-      (effects (font (size 1.27 1.27)) hide)
-    )
-    (pin "1")
-    (instances
-      (project "version_1"
-        (path "/23ba0750-4a55-4d50-828b-749cc0fbb8c8"
-          (reference "#PWR010") (unit 1)
-        )
-        (path "/23ba0750-4a55-4d50-828b-749cc0fbb8c8/79f7122c-c2a5-4829-b847-ff54a5199600"
-          (reference "#PWR0200") (unit 1)
-        )
-        (path "/23ba0750-4a55-4d50-828b-749cc0fbb8c8/d2110296-333c-46f5-b5da-c8cbeafe02ed"
-          (reference "#PWR0201") (unit 1)
-        )
-        (path "/23ba0750-4a55-4d50-828b-749cc0fbb8c8/1b8f704b-b129-4c22-a423-d346d579d0e5"
-          (reference "#PWR0202") (unit 1)
-        )
-        (path "/23ba0750-4a55-4d50-828b-749cc0fbb8c8/0734ecc9-bf55-4847-b598-21bbdec71699"
-          (reference "#PWR0203") (unit 1)
-        )
-      )

Commit message: encoder power fliping
Connections:
- net ENC_PWR_1 renamed ENC_PWR_P
- net ENC_PWR_2 renamed ENC_PWR_G
Changed lines of the file:
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@@
     (effects (font (size 1.27 1.27)) (justify left bottom))
   )
-  (global_label "ENC_PWR_2" (shape input) (at 148.59 90.17 180) (fields_autoplaced)
+  (global_label "ENC_PWR_G" (shape input) (at 148.59 90.17 180) (fields_autoplaced)
     (effects (font (size 1.27 1.27)) (justify right))
-    (property "Intersheetrefs" "${INTERSHEET_REFS}" (at 134.7986 90.17 0)
+    (property "Intersheetrefs" "${INTERSHEET_REFS}" (at 134.7381 90.17 0)
       (effects (font (size 1.27 1.27)) (justify right) hide)
     )
   )
-  (global_label "ENC_PWR_1" (shape input) (at 148.59 74.93 180) (fields_autoplaced)
+  (global_label "ENC_PWR_P" (shape input) (at 148.59 74.93 180) (fields_autoplaced)
     (effects (font (size 1.27 1.27)) (justify right))
-    (property "Intersheetrefs" "${INTERSHEET_REFS}" (at 134.7986 74.93 0)
+    (property "Intersheetrefs" "${INTERSHEET_REFS}" (at 134.7381 74.93 0)
       (effects (font (size 1.27 1.27)) (justify right) hide)
     )
