File: H_bridge.kicad_sch (KiCad schematic)
At the start: 11 parts, among them CN1 B6B-PH-K-S(LF)(SN), U13 DRV8870DDA

Commit message: big layout changes
Parts:
- removed C1: 100n, Capacitor_SMD:C_0603_1608Metric_Pad1.08x0.95mm_HandSolder, symbol Device:C_Small
- removed C10 (x2): 22u, Capacitor_SMD:C_0805_2012Metric_Pad1.18x1.45mm_HandSolder, symbol Device:C

Commit message: exported
Parts:
- added Q?: AO3400A, Package_TO_SOT_SMD:SOT-23, symbol Transistor_FET:AO3400A
- U13: LCSC (none) -> C86590
Changed lines of the file:
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@@
+    )
+  )
+  (symbol (lib_id "Transistor_FET:AO3400A") (at 86.36 156.21 0) (unit 1)
+    (in_bom yes) (on_board yes) (dnp no)
+    (property "Reference" "Q?" (at 92.71 155.575 0)
+      (effects (font (size 1.27 1.27)) (justify left))
+    )
+    (property "Value" "AO3400A" (at 92.71 158.115 0)
+      (effects (font (size 1.27 1.27)) (justify left))
+    )
+    (property "Footprint" "Package_TO_SOT_SMD:SOT-23" (at 91.44 158.115 0)
+      (effects (font (size 1.27 1.27) italic) (justify left) hide)
+    )
+    (property "Datasheet" "http://www.aosmd.com/pdfs/datasheet/AO3400A.pdf" (at 86.36 156.21 0)
+      (effects (font (size 1.27 1.27)) (justify left) hide)
+    )
+    (property "JLCPCB Part#" "C20917" (at 86.36 156.21 0)
+      (effects (font (size 1.27 1.27)) hide)
+    )
+    (pin "1")
+    (pin "2")
+    (pin "3")
+    (instances
+      (project "version_1"
+        (path "/23ba0750-4a55-4d50-828b-749cc0fbb8c8"
+          (reference "Q?") (unit 1)
+        )
+        (path "/23ba0750-4a55-4d50-828b-749cc0fbb8c8/79f7122c-c2a5-4829-b847-ff54a5199600"
+          (reference "Q6") (unit 1)
+        )
+        (path "/23ba0750-4a55-4d50-828b-749cc0fbb8c8/9789521c-7f58-473a-9dd2-6c6a71290f6c"
+          (reference "Q21") (unit 1)
+        )
+        (path "/23ba0750-4a55-4d50-828b-749cc0fbb8c8/d2110296-333c-46f5-b5da-c8cbeafe02ed"
+          (reference "Q21") (unit 1)
+        )
+        (path "/23ba0750-4a55-4d50-828b-749cc0fbb8c8/1b8f704b-b129-4c22-a423-d346d579d0e5"
+          (reference "Q21") (unit 1)
+        )
+        (path "/23ba0750-4a55-4d50-828b-749cc0fbb8c8/0734ecc9-bf55-4847-b598-21bbdec71699"
+          (reference "Q21") (unit 1)
+        )
+      )
     )
   )
@@
       (effects (font (size 1.27 1.27)) hide)
     )
+    (property "LCSC" "C86590" (at 113.03 83.82 0)
+      (effects (font (size 1.27 1.27)) hide)
+    )

Commit message: 4 layer
Parts:
- removed Q?: AO3400A, Package_TO_SOT_SMD:SOT-23, symbol Transistor_FET:AO3400A
- added R26: 0.27, Resistor_SMD:R_0603_1608Metric_Pad0.98x0.95mm_HandSolder, symbol Device:R
Connections:
- net GND: now also R26.2; no longer U13.7 (ISEN)
- new net: R26.1, U13.7 (ISEN)
Other:
- note added: "1.85A limmit"
