File: version_1.kicad_pcb (KiCad board)
At the start: 2 copper layers, 100 x 110 mm, 101 parts, among them CN1 B6B-PH-K-S(LF)(SN), CN2 B6B-PH-K-S(LF)(SN), CN3 B6B-PH-K-S(LF)(SN), CN4 B6B-PH-K-S(LF)(SN), M5 Motor_Servo_JR, M6 Motor_Servo_JR, M7 Motor_Servo_JR, M8 Motor_Servo_JR, Q17 AO3401A, Q18 AO3401A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

Commit message: tetris
Parts:
- moved JP1 57.6 mm to (82.5, 44.5), turned to 0 degrees
- moved C15 53.0 mm to (91.4, 43.2)
- moved R25 53.0 mm to (91.3, 45.2)
- moved R26 53.0 mm to (87.7, 45.2)
- moved C60 46.6 mm to (147.6, 46.0), turned to -90 degrees
- moved C61 46.0 mm to (149.5, 46.0), turned to -90 degrees
- moved C59 46.0 mm to (154.5, 46.0), turned to -90 degrees
- moved C8 46.0 mm to (152.0, 46.0), turned to -90 degrees
- moved JP4 40.3 mm to (134.0, 38.0)
- moved Q21 11.0 mm to (25.1, 103.6)
- moved Q23 11.0 mm to (25.1, 107.3)
- moved Q22 11.0 mm to (25.1, 100.0)
- moved Q24 11.0 mm to (25.1, 92.8)
- moved Q25 11.0 mm to (25.1, 96.4)
- moved U18 10.4 mm to (23.5, 87.6)
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Connections:
- U1 pad 14: /ENCODER1 -> /ENCODER5
- U1 pad 15: /ENCODER2 -> /ENCODER6
- U1 pad 19: /ENCODER5 -> /ENCODER1
- U1 pad 20: /ENCODER6 -> /ENCODER2
- U1 pad 21: /MR3 -> /ML1
- U1 pad 22: /ML3 -> /MR1
- U1 pad 24: /MR2 -> /ML2
- U1 pad 25: /ML2 -> /MR2
- U1 pad 26: /MR1 -> /ML3
- U1 pad 27: /ML1 -> /MR3
- U1 pad 31: /MR4 -> /ML4
- U1 pad 32: /ML4 -> /MR4
Routing:
- net +5V: track 58.3 -> 167.6 mm, vias 2 -> 10
- net Net-(D5-A): track 6.43 -> 71.5 mm, vias 0 -> 4
- net Net-(U1-GPIO28_ADC2): track 7.66 -> 63.8 mm, vias 0 -> 2
- net VCC: track 256.1 -> 303.0 mm, vias 12 -> 15
- net /ENCODER4: track 32.9 -> 71.2 mm, vias 4 -> 8
- net /PWM_CLK: track 67.6 -> 104.7 mm
- net /ENCODER3: track 32.1 -> 67.5 mm, vias 4 -> 7
- net /PWM_CS: track 74.1 -> 108.3 mm, vias 0 -> 2
- net /ENCODER2: track 18.9 -> 52.6 mm, vias 2 -> 4
- net /ENCODER8: track 16.5 -> 48.7 mm, vias 2 -> 4
- net /PWM_DATA: track 73.1 -> 104.7 mm, vias 2 -> 0
- net /ENCODER7: track 16.0 -> 47.4 mm, vias 2 -> 4
- net +3.3V: track 109.1 -> 88.6 mm, vias 2 -> 4
- net /ENCODER1: track 32.1 -> 51.9 mm
- net /ENCODER5: track 32.1 -> 51.8 mm, vias 4 -> 6
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Other:
- board size 100 x 110 mm -> 100 x 100 mm
- board text added: "S"

Commit message: cleanup
Parts:
- moved C60 53.7 mm to (94.6, 36.8), turned to 180 degrees
- moved C8 49.3 mm to (102.9, 41.9), turned to 0 degrees
- moved JP4 37.3 mm to (97.0, 43.0)
- moved C59 36.5 mm to (118.1, 48.9)
- moved C61 35.2 mm to (114.3, 45.1), turned to 180 degrees
- moved Q21 1.39 mm to (25.1, 105.0)
- moved Q22 1.39 mm to (25.1, 101.4)
- moved Q23 1.39 mm to (25.1, 108.7)
- moved Q25 1.39 mm to (25.1, 97.8)
- moved Q24 1.38 mm to (25.1, 94.2)
- moved C6 1.27 mm to (89.5, 48.3)
- moved JP1 0.84 mm to (82.0, 43.8), turned to 180 degrees
- moved C5 0.64 mm to (79.4, 48.2)
- moved U2 0.33 mm to (99.3, 59.1)
Routing:
- net 1S: track 104.1 -> 185.6 mm, vias 0 -> 2
- net Net-(U1-GPIO28_ADC2): track 63.8 -> 83.8 mm
- net Linear 5V: track 3.57 -> 21.5 mm
- net VCC: track 303.0 -> 315.7 mm, vias 15 -> 17
- net Net-(D5-A): track 71.5 -> 83.8 mm
- net +5V: track 167.6 -> 178.9 mm, vias 10 -> 11
- net /ENCODER6: track 48.5 -> 55.5 mm
- net ENC_PWR_P: track 82.1 -> 86.1 mm
- net Net-(JP4-A): track 22.3 -> 25.5 mm
- net /Untitled Sheet7/PWR: track 23.1 -> 24.8 mm
- net /SCL: track 43.5 -> 45.1 mm
- net /Untitled Sheet7/PWM: track 32.1 -> 33.3 mm
- net /PWM_CLK: track 104.7 -> 103.9 mm
- net Net-(D1-A): track 126.8 -> 126.0 mm
- net /MR1: track 20.4 -> 19.8 mm
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- removed copper zone on F.Cu, net (none)
- removed copper zone on F.Cu, net Net-(F1-Pad1)
- removed copper zone on B.Cu, net VCC
- removed copper zone on F.Cu, net VCC

Commit message: delt with errors
Routing:
- net /ENCODER3: track 67.5 -> 58.9 mm, vias 7 -> 6
- net ENC_PWR_G: track 89.1 -> 82.5 mm
- net GND: track 184.8 -> 189.0 mm, vias 66 -> 171
- net ENC_PWR_P: track 86.1 -> 83.1 mm, vias 7 -> 6
- net /ENCODER4: track 71.2 -> 69.1 mm
- net Net-(D5-A): track 83.8 -> 84.6 mm
- net /ENCODER2: track 52.6 -> 51.9 mm
- net Net-(U1-GPIO28_ADC2): track 83.8 -> 84.3 mm
Other:
- outline, holes or cut-outs redrawn
- board text removed: "LED1"
- board text removed: "LED2"

Commit message: wearninigs
Routing:
- net ENC_PWR_G: track 82.5 -> 80.7 mm
- net Net-(D1-A): track 126.0 -> 124.7 mm
- net +3.3V: track 88.6 -> 87.5 mm
- net 1S: track 185.6 -> 184.6 mm
- net /ENCODER2: track 51.9 -> 50.9 mm
- net +5V: track 178.9 -> 178.2 mm
- net VCC: track 315.7 -> 315.1 mm, vias 17 -> 16
- net ENC_PWR_P: track 83.1 -> 82.8 mm, vias 6 -> 5
- net /ENCODER6: track 55.5 -> 55.4 mm, vias 6 -> 4
- net GND: vias 171 -> 168
- net /ENCODER5: vias 6 -> 4
- net /ENCODER4: vias 8 -> 6

Commit message: mostly done
Parts:
- moved Q21 0.34 mm to (25.4, 105.0)
- moved Q22 0.34 mm to (25.4, 101.4)
- moved Q23 0.34 mm to (25.4, 108.7)
- moved Q24 0.34 mm to (25.4, 94.2)
- moved Q25 0.34 mm to (25.4, 97.8)
Other:
- board text added: "Robotyka v2 2024-05-31"
- board text added: "SN:"
- board text removed: "designed by: Michał Pietrzak"
- board text removed: "for: Fundacja Adamed www.fundacjaadamed.pl"
- board text removed: "serial no:"

Commit message: 4 layer
Parts:
- removed F1: DFN, Fuse:Fuse_1210_3225Metric_Pad1.42x2.65mm_HandSolder
- removed U2: SS-12D10L5, footprint:SW-TH_SS-12D10L5
- added F2: SMD2920B500TF, footprint:F2920, F.Cu at (116.8, 63.5)
- added R10: 0.27, Resistor_SMD:R_0603_1608Metric_Pad0.98x0.95mm_HandSolder, F.Cu at (35.6, 27.3)
- added R5: 100k, Resistor_SMD:R_0603_1608Metric_Pad0.98x0.95mm_HandSolder, F.Cu at (91.4, 52.1)
- added R6: 100k, Resistor_SMD:R_0603_1608Metric_Pad0.98x0.95mm_HandSolder, F.Cu at (91.4, 48.3)
- added R7: 0.27, Resistor_SMD:R_0603_1608Metric_Pad0.98x0.95mm_HandSolder, F.Cu at (81.3, 27.3)
- added R8: 0.27, Resistor_SMD:R_0603_1608Metric_Pad0.98x0.95mm_HandSolder, F.Cu at (66.7, 26.7)
- added R9: 0.27, Resistor_SMD:R_0603_1608Metric_Pad0.98x0.95mm_HandSolder, F.Cu at (50.8, 27.3)
- added U7: 2AD1T1A2M2QES, footprint:SW-TH_2AD1T1A2M2QES, F.Cu at (97.8, 57.8)
- moved C13 9.05 mm to (106.0, 54.0), turned to -90 degrees
- moved D4 1.59 mm to (108.6, 54.0), turned to 90 degrees
- moved R1 1.54 mm to (108.6, 58.4), turned to 90 degrees
- moved C30 1.51 mm to (103.5, 54.0), turned to -90 degrees
- moved R17 1.15 mm to (115.6, 99.4)
- moved D3 0.90 mm to (115.6, 102.7)
- moved D1 0.64 mm to (116.2, 118.1)
- moved R20 0.64 mm to (116.2, 115.6)
- moved C6 0.63 mm to (88.9, 48.3), turned to -90 degrees
- moved CN3 0.07 mm to (51.9, 22.2)
Connections:
- Q21 pad 1: VCC -> Net-(Q21-G)
- Q22 pad 1: VCC -> Net-(Q21-G)
- Q23 pad 1: VCC -> Net-(Q21-G)
- Q24 pad 1: VCC -> Net-(Q21-G)
- Q25 pad 1: VCC -> Net-(Q21-G)
- U13 pad 7: GND -> Net-(U13-ISEN)
- U15 pad 7: GND -> Net-(U15-ISEN)
- U16 pad 7: GND -> Net-(U16-ISEN)
- U17 pad 7: GND -> Net-(U17-ISEN)
Routing:
- net Net-(Q21-G): track 0.00 -> 120.6 mm, vias 0 -> 10
- net VCC: track 315.1 -> 204.5 mm, vias 16 -> 6
- net Net-(F2-Pad2): track 0.00 -> 29.1 mm
- net Net-(F1-Pad1): track 14.7 -> 0.00 mm
- net Net-(U16-OUT1): track 19.4 -> 9.72 mm
- net Net-(U13-OUT1): track 19.4 -> 9.92 mm
- net Net-(U15-OUT1): track 19.4 -> 10.1 mm
- net GND: track 189.0 -> 182.3 mm, vias 168 -> 177
- net ENC_PWR_G: track 80.7 -> 76.1 mm
- net Net-(U15-ISEN): track 0.00 -> 3.20 mm
- net Net-(U16-ISEN): track 0.00 -> 3.02 mm
- net Net-(U17-ISEN): track 0.00 -> 2.89 mm
- net Net-(U13-ISEN): track 0.00 -> 2.84 mm
- net +3.3V: track 87.5 -> 89.6 mm
- net ENC_PWR_P: track 82.8 -> 81.6 mm
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- added copper zone on In1.Cu, net GND
- added copper zone on In2.Cu, net GND
Other:
- outline, holes or cut-outs redrawn
- copper layers 2 -> 4
- board text added: "3v3"
- board text added: "Flipped Cell!"
- board text added: "GND"
- board text added: "I2C Qwiic"
